File: packages/esp32s3/layouts/ref-esp32s3/esp32s3.kicad_pcb (KiCad board)
At the start: 2 copper layers, 6 parts

Commit message: fixed
Connections:
- net in renamed input
Changed lines of the file:
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@@
     )
     (net 0 "")
-    (net 1 "in")
+    (net 1 "input")
     (net 2 "io4")
     (net 3 "io5")
@@
             (size 0.57 0.54)
             (layers "F.Cu" "F.Mask" "F.Paste")
-            (net 1 "in")
+            (net 1 "input")
         )
         (embedded_fonts no)
@@
             (size 1.05 0.7)
             (layers "F.Cu" "F.Mask" "F.Paste")
-            (net 1 "in")
+            (net 1 "input")
             (pintype "stereo")
         )
@@
             (size 1.05 0.7)
             (layers "F.Cu" "F.Mask" "F.Paste")
-            (net 1 "in")
-            (pintype "stereo")
-        )
+            (net 1 "input")
+            (pintype "stereo")
+        )
