File: packages/ti-ina232/layouts/default/default.kicad_pcb (KiCad board)
At the start: 2 copper layers, 3 parts

Commit message: fixed?
Parts:
- C1: footprint atopile:C0402-b3ef17 -> Samsung_Electro_Mechanics_CL05B104KO5NNNC:C0402
- R1: value 100Ω ±1% 250mW -> 0Ω 250mW; footprint atopile:R1206-bdb864 -> UNI_ROYAL_1206W4F0000T5E:R1206
- U1: footprint atopile:SOT-23-8_L2.9-W1.6-P0.65-LS2.8-BR-f3715a -> TEXAS_INSTRUMENTS_INA232AIDDFR:SOT-23-8_L2.9-W1.6-P0.65-LS2.8-BR
