File: packages/ti-ina232/layouts/test/test.kicad_pcb (KiCad board)
At the start: 2 copper layers, 12 parts

Commit message: fixed?
Parts:
- C1, C2, C3, C4: footprint atopile:C0402-b3ef17 -> Samsung_Electro_Mechanics_CL05B104KO5NNNC:C0402
- R1: value 750mΩ ±1% 250mW -> 800mΩ ±1% 250mW; footprint atopile:R1206-bdb864 -> FOJAN_FRL1206FR800TS:R1206
- R2: value 70mΩ ±1% 1W -> 70mΩ ±1% 500mW; footprint atopile:R1206-bdb864 -> YAGEO_PE1206FRM7W0R07L:R1206
- R3: footprint atopile:R1206-bdb864 -> Milliohm_HoYLR1206_1W_25mR_1:R1206
- R4: value 8mΩ ±1% 1W -> 7mΩ ±1% 1W; footprint atopile:R1206-bdb864 -> Milliohm_HoLLR1206_1W_7mR_1:R1206
- U1, U2, U3, U4: footprint atopile:SOT-23-8_L2.9-W1.6-P0.65-LS2.8-BR-f3715a -> TEXAS_INSTRUMENTS_INA232AIDDFR:SOT-23-8_L2.9-W1.6-P0.65-LS2.8-BR
Connections:
- C1 pad 2: gnd-1 -> gnd-2
- C2 pad 2: gnd-1 -> gnd-2
- C3 pad 2: gnd-1 -> gnd-2
- C4 pad 2: gnd-1 -> gnd-2
- R2 pad 1: gnd-2 -> gnd
- R2 pad 2: gnd -> gnd-1
- U1 pad 3: gnd-1 -> gnd-2
- U1 pad 7: gnd-1 -> gnd-2
- U2 pad 1: gnd-2 -> gnd
- U2 pad 2: gnd -> gnd-1
- U2 pad 3: gnd-1 -> gnd-2
- U3 pad 3: gnd-1 -> gnd-2
- U4 pad 3: gnd-1 -> gnd-2
Routing:
- net gnd-2: track 2.13 -> 9.38 mm
- net gnd-1: track 9.38 -> 3.25 mm
- net gnd: track 3.25 -> 2.13 mm
